File: PCB/FPGA_DENDY_SE.sch (EAGLE design)
At the start: 138 parts, among them CN1 DENDY60PINSLOT, J1 NTSC/PAL, J2 DENDY, Q1 14.318 MHz, Q2 17.734 MHz, U1 EP1C3T100C8N, U10 OPA2134U, U11 SN74LVC2G34DBVR, U12 THS7314DR, U13 74LS373WMSO20, U14 SN74LVC1G125DBVR, U15 74LVC1G04GV, U16 SN74LVC1G3157, U2 EPCS4, U3 SN74LVC8T245, U4 SN74LVC8T245, U5 SN74LVC1G240DCKR, U6 SN74LVC1G240DCKR, U7 SN74LVC1G240DCKR, U8 SN74LVC1G240DCKR, X1 057-010-1

Commit message: Add files via upload
Parts:
- U5, U6, U7, U8: value SN74LVC1G240DCKR -> SN74LVC1G240DBVR; device SN74LVC1G240DCKR:SN74LVC1G240DCKR -> SN74LVC1G240DBVR:SN74LVC1G240DBVR
Connections:
- net /IN0: now also U6./OE, U8./OE; no longer U5./OE, U7./OE
- net /IN1: now also U5./OE, U7./OE; no longer U6./OE, U8./OE
- net D0: now also U5.Y, U6.Y; no longer U7.Y, U8.Y
- net JOYDATA1: now also U6.A; no longer U7.A
- net JOYDATA2: now also U5.A; no longer U8.A
- net M2_FPGA: now also U7.A, U8.A; no longer U5.A, U6.A
- net SCK1: now also U8.Y; no longer U5.Y
- net SCK2: now also U7.Y; no longer U6.Y
Other:
- moved on the sheet: U5, U6, U7, U8
Changed lines of the file:
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@@
 <?xml version="1.0" encoding="utf-8"?>
 <!DOCTYPE eagle SYSTEM "eagle.dtd">
-<eagle version="9.4.2">
+<eagle version="9.6.2">
 <drawing>
 <settings>
@@
 <part name="C6" library="rcl_my" deviceset="C-EU" device="C0805" package3d_urn="urn:adsk.eagle:package:23617/2" value="0.01uF"/>
 <part name="GND50" library="supply1" library_urn="urn:adsk.eagle:library:371" deviceset="GND" device=""/>
-<part name="U5" library="SN74LVC1G240DCKR" deviceset="SN74LVC1G240DCKR" device="" value="SN74LVC1G240DCKR"/>
-<part name="U6" library="SN74LVC1G240DCKR" deviceset="SN74LVC1G240DCKR" device="" value="SN74LVC1G240DCKR"/>
-<part name="U7" library="SN74LVC1G240DCKR" deviceset="SN74LVC1G240DCKR" device="" value="SN74LVC1G240DCKR"/>
-<part name="U8" library="SN74LVC1G240DCKR" deviceset="SN74LVC1G240DCKR" device="" value="SN74LVC1G240DCKR"/>
 <part name="RN1" library="resistor-dil" library_urn="urn:adsk.eagle:library:342" deviceset="4R-N" device="0603-ARC" package3d_urn="urn:adsk.eagle:package:24926/1" value="22"/>
 <part name="RN2" library="resistor-dil" library_urn="urn:adsk.eagle:library:342" deviceset="4R-N" device="0603-ARC" package3d_urn="urn:adsk.eagle:package:24926/1" value="22"/>
@@
 <part name="R25" library="rcl" library_urn="urn:adsk.eagle:library:334" deviceset="R-EU_" device="R0805" package3d_urn="urn:adsk.eagle:package:23553/2" value="51"/>
 <part name="JP1" library="jumper" library_urn="urn:adsk.eagle:library:252" deviceset="JP4QE" device="" package3d_urn="urn:adsk.eagle:package:15451/1"/>
+<part name="U5" library="SN74LVC1G240DBVR" deviceset="SN74LVC1G240DBVR" device="" value="SN74LVC1G240DBVR"/>
+<part name="U6" library="SN74LVC1G240DBVR" deviceset="SN74LVC1G240DBVR" device="" value="SN74LVC1G240DBVR"/>
+<part name="U7" library="SN74LVC1G240DBVR" deviceset="SN74LVC1G240DBVR" device="" value="SN74LVC1G240DBVR"/>
+<part name="U8" library="SN74LVC1G240DBVR" deviceset="SN74LVC1G240DBVR" device="" value="SN74LVC1G240DBVR"/>
 </parts>
 <sheets>
@@
 </instance>
 <instance part="GND50" gate="1" x="48.26" y="-91.44" smashed="yes" rot="R270"/>
-<instance part="U5" gate="A" x="165.1" y="38.1" smashed="yes">
-<attribute name="NAME" x="163.576" y="49.26" size="2.0828" layer="95" ratio="10" rot="SR0"/>
-<attribute name="VALUE" x="152.4" y="23.94" size="2.0828" layer="96" ratio="10" rot="SR0"/>
-</instance>
-<instance part="U6" gate="A" x="165.1" y="7.62" smashed="yes">
-<attribute name="NAME" x="163.322" y="18.78" size="2.0828" layer="95" ratio="10" rot="SR0"/>
-<attribute name="VALUE" x="152.4" y="-6.54" size="2.0828" layer="96" ratio="10" rot="SR0"/>
-</instance>
-<instance part="U7" gate="A" x="165.1" y="-22.86" smashed="yes">
-<attribute name="NAME" x="163.322" y="-11.7" size="2.0828" layer="95" ratio="10" rot="SR0"/>
-<attribute name="VALUE" x="152.4" y="-37.02" size="2.0828" layer="96" ratio="10" rot="SR0"/>
-</instance>
-<instance part="U8" gate="A" x="165.1" y="-53.34" smashed="yes">
-<attribute name="NAME" x="163.322" y="-42.18" size="2.0828" layer="95" ratio="10" rot="SR0"/>
-<attribute name="VALUE" x="152.4" y="-67.5" size="2.0828" layer="96" ratio="10" rot="SR0"/>
-</instance>
 <instance part="RN1" gate="A" x="-327.66" y="144.78" smashed="yes">
 <attribute name="VALUE" x="-323.088" y="141.732" size="1.778" layer="96"/>
@@
 <attribute name="VALUE" x="-248.285" y="-88.9" size="1.778" layer="96" rot="R90"/>
 </instance>
+<instance part="U5" gate="A" x="165.1" y="-53.34" smashed="yes">
+<attribute name="NAME" x="163.068" y="-42.18" size="2.0828" layer="95" ratio="10" rot="SR0"/>
+<attribute name="VALUE" x="152.4" y="-67.5" size="2.0828" layer="96" ratio="10" rot="SR0"/>
+</instance>
+<instance part="U6" gate="A" x="165.1" y="-22.86" smashed="yes">
+<attribute name="NAME" x="163.068" y="-11.7" size="2.0828" layer="95" ratio="10" rot="SR0"/>
+<attribute name="VALUE" x="152.4" y="-37.02" size="2.0828" layer="96" ratio="10" rot="SR0"/>
+</instance>
+<instance part="U7" gate="A" x="165.1" y="7.62" smashed="yes">
+<attribute name="NAME" x="163.068" y="18.78" size="2.0828" layer="95" ratio="10" rot="SR0"/>
+<attribute name="VALUE" x="152.4" y="-6.54" size="2.0828" layer="96" ratio="10" rot="SR0"/>
+</instance>
+<instance part="U8" gate="A" x="165.1" y="38.1" smashed="yes">
+<attribute name="NAME" x="163.068" y="49.26" size="2.0828" layer="95" ratio="10" rot="SR0"/>
+<attribute name="VALUE" x="152.4" y="23.94" size="2.0828" layer="96" ratio="10" rot="SR0"/>
+</instance>
 </instances>
 <busses>
@@
 </segment>
 <segment>
-<pinref part="U5" gate="A" pin="VCC"/>
 <wire x1="182.88" y1="45.72" x2="198.12" y2="45.72" width="0.1524" layer="91"/>
 <wire x1="198.12" y1="45.72" x2="198.12" y2="76.2" width="0.1524" layer="91"/>
-<pinref part="U6" gate="A" pin="VCC"/>
 <wire x1="198.12" y1="76.2" x2="198.12" y2="81.28" width="0.1524" layer="91"/>
 <wire x1="182.88" y1="15.24" x2="198.12" y2="15.24" width="0.1524" layer="91"/>
 <wire x1="198.12" y1="15.24" x2="198.12" y2="30.48" width="0.1524" layer="91"/>
 <junction x="198.12" y="45.72"/>
-<pinref part="U7" gate="A" pin="VCC"/>
 <wire x1="198.12" y1="30.48" x2="198.12" y2="45.72" width="0.1524" layer="91"/>
 <wire x1="182.88" y1="-15.24" x2="198.12" y2="-15.24" width="0.1524" layer="91"/>
 <wire x1="198.12" y1="-15.24" x2="198.12" y2="15.24" width="0.1524" layer="91"/>
 <junction x="198.12" y="15.24"/>
-<pinref part="U8" gate="A" pin="VCC"/>
 <wire x1="182.88" y1="-45.72" x2="198.12" y2="-45.72" width="0.1524" layer="91"/>
 <wire x1="198.12" y1="-30.48" x2="198.12" y2="-15.24" width="0.1524" layer="91"/>
@@
 <junction x="198.12" y="76.2"/>
 <junction x="198.12" y="-45.72"/>
+<pinref part="U5" gate="A" pin="VCC"/>
+<pinref part="U6" gate="A" pin="VCC"/>
+<pinref part="U7" gate="A" pin="VCC"/>
+<pinref part="U8" gate="A" pin="VCC"/>
 </segment>
 <segment>
@@
 <segment>
 <label x="193.04" y="-53.34" size="1.778" layer="95"/>
-<pinref part="U7" gate="A" pin="Y"/>
 <wire x1="182.88" y1="-22.86" x2="187.96" y2="-22.86" width="0.1524" layer="91"/>
-<pinref part="U8" gate="A" pin="Y"/>
 <wire x1="187.96" y1="-22.86" x2="187.96" y2="-53.34" width="0.1524" layer="91"/>
 <wire x1="187.96" y1="-53.34" x2="182.88" y2="-53.34" width="0.1524" layer="91"/>
 <wire x1="198.12" y1="-53.34" x2="187.96" y2="-53.34" width="0.1524" layer="91"/>
 <junction x="187.96" y="-53.34"/>
+<pinref part="U5" gate="A" pin="Y"/>
+<pinref part="U6" gate="A" pin="Y"/>
 </segment>
 </net>
@@
 <wire x1="147.32" y1="-30.48" x2="132.08" y2="-30.48" width="0.1524" layer="91"/>
 <label x="134.62" y="-30.48" size="1.778" layer="95"/>
-<pinref part="U7" gate="A" pin="A"/>
+<pinref part="U6" gate="A" pin="A"/>
 </segment>
 </net>
@@
 <wire x1="147.32" y1="-60.96" x2="132.08" y2="-60.96" width="0.1524" layer="91"/>
 <label x="134.62" y="-60.96" size="1.778" layer="95"/>
-<pinref part="U8" gate="A" pin="A"/>
+<pinref part="U5" gate="A" pin="A"/>
 </segment>
 </net>
@@
 <wire x1="193.04" y1="7.62" x2="182.88" y2="7.62" width="0.1524" layer="91"/>
 <label x="185.42" y="7.62" size="1.778" layer="95"/>
-<pinref part="U6" gate="A" pin="Y"/>
+<pinref part="U7" gate="A" pin="Y"/>
 </segment>
 </net>
@@
 <wire x1="193.04" y1="38.1" x2="182.88" y2="38.1" width="0.1524" layer="91"/>
 <label x="185.42" y="38.1" size="1.778" layer="95"/>
-<pinref part="U5" gate="A" pin="Y"/>
+<pinref part="U8" gate="A" pin="Y"/>
 </segment>
 </net>
@@
 <wire x1="147.32" y1="30.48" x2="132.08" y2="30.48" width="0.1524" layer="91"/>
 <label x="134.62" y="30.48" size="1.778" layer="95"/>
-<pinref part="U5" gate="A" pin="A"/>
+<pinref part="U8" gate="A" pin="A"/>
 </segment>
 <segment>
 <wire x1="147.32" y1="0" x2="132.08" y2="0" width="0.1524" layer="91"/>
 <label x="134.62" y="0" size="1.778" layer="95"/>
-<pinref part="U6" gate="A" pin="A"/>
+<pinref part="U7" gate="A" pin="A"/>
 </segment>
 <segment>
@@
 <wire x1="147.32" y1="45.72" x2="132.08" y2="45.72" width="0.1524" layer="91"/>
 <label x="134.62" y="45.72" size="1.778" layer="95"/>
-<pinref part="U5" gate="A" pin="/OE"/>
+<pinref part="U8" gate="A" pin="/OE"/>
 </segment>
 <segment>
 <wire x1="147.32" y1="-15.24" x2="132.08" y2="-15.24" width="0.1524" layer="91"/>
 <label x="134.62" y="-15.24" size="1.778" layer="95"/>
-<pinref part="U7" gate="A" pin="/OE"/>
+<pinref part="U6" gate="A" pin="/OE"/>
 </segment>
 </net>
@@
 <wire x1="147.32" y1="15.24" x2="132.08" y2="15.24" width="0.1524" layer="91"/>
 <label x="134.62" y="15.24" size="1.778" layer="95"/>
-<pinref part="U6" gate="A" pin="/OE"/>
+<pinref part="U7" gate="A" pin="/OE"/>
 </segment>
 <segment>
 <wire x1="147.32" y1="-45.72" x2="132.08" y2="-45.72" width="0.1524" layer="91"/>
 <label x="134.62" y="-45.72" size="1.778" layer="95"/>
-<pinref part="U8" gate="A" pin="/OE"/>
+<pinref part="U5" gate="A" pin="/OE"/>
 </segment>
 </net>

Commit message: Add files via upload
Connections:
- net DENDY renamed /DENDY
- net PAL renamed /PAL
Changed lines of the file:
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@@
-</segment>
-</net>
-<net name="DENDY" class="0">
-<segment>
-<pinref part="J2" gate="A" pin="1"/>
-<wire x1="-111.76" y1="68.58" x2="-129.54" y2="68.58" width="0.1524" layer="91"/>
-<label x="-127" y="68.58" size="1.778" layer="95"/>
-</segment>
-<segment>
-<wire x1="-45.72" y1="22.86" x2="-60.96" y2="22.86" width="0.1524" layer="91"/>
-<label x="-58.42" y="22.86" size="1.778" layer="95"/>
-<pinref part="U1" gate="G$1" pin="IO3"/>
 </segment>
 </net>
@@
 <pinref part="Q2" gate="G$1" pin="OUT"/>
 <wire x1="-50.8" y1="-109.22" x2="-55.88" y2="-109.22" width="0.1524" layer="91"/>
-</segment>
-</net>
-<net name="PAL" class="0">
-<segment>
-<pinref part="J1" gate="A" pin="1"/>
-<wire x1="-111.76" y1="78.74" x2="-129.54" y2="78.74" width="0.1524" layer="91"/>
-<label x="-127" y="78.74" size="1.778" layer="95"/>
-</segment>
-<segment>
-<wire x1="-45.72" y1="27.94" x2="-60.96" y2="27.94" width="0.1524" layer="91"/>
-<label x="-58.42" y="27.94" size="1.778" layer="95"/>
-<pinref part="U1" gate="G$1" pin="IO1"/>
-</segment>
-<segment>
-<wire x1="-17.78" y1="-99.06" x2="-50.8" y2="-99.06" width="0.1524" layer="91"/>
-<label x="-48.26" y="-99.06" size="1.778" layer="95"/>
-<pinref part="U16" gate="G$1" pin="S"/>
-<wire x1="-17.78" y1="-99.06" x2="-17.78" y2="-106.68" width="0.1524" layer="91"/>
 </segment>
 </net>
@@
 </segment>
 </net>
+<net name="/PAL" class="0">
+<segment>
+<pinref part="J1" gate="A" pin="1"/>
+<wire x1="-111.76" y1="78.74" x2="-129.54" y2="78.74" width="0.1524" layer="91"/>
+<label x="-127" y="78.74" size="1.778" layer="95"/>
+</segment>
+<segment>
+<wire x1="-45.72" y1="27.94" x2="-60.96" y2="27.94" width="0.1524" layer="91"/>
+<label x="-58.42" y="27.94" size="1.778" layer="95"/>
+<pinref part="U1" gate="G$1" pin="IO1"/>
+</segment>
+<segment>
+<wire x1="-17.78" y1="-99.06" x2="-50.8" y2="-99.06" width="0.1524" layer="91"/>
+<label x="-48.26" y="-99.06" size="1.778" layer="95"/>
+<pinref part="U16" gate="G$1" pin="S"/>
+<wire x1="-17.78" y1="-99.06" x2="-17.78" y2="-106.68" width="0.1524" layer="91"/>
+</segment>
+</net>
+<net name="/DENDY" class="0">
+<segment>
+<pinref part="J2" gate="A" pin="1"/>
+<wire x1="-111.76" y1="68.58" x2="-129.54" y2="68.58" width="0.1524" layer="91"/>
+<label x="-127" y="68.58" size="1.778" layer="95"/>
+</segment>
+<segment>
+<wire x1="-45.72" y1="22.86" x2="-60.96" y2="22.86" width="0.1524" layer="91"/>
+<label x="-58.42" y="22.86" size="1.778" layer="95"/>
+<pinref part="U1" gate="G$1" pin="IO3"/>
+</segment>
+</net>

Commit message: Add files via upload
Parts:
- added RN11: 1k, resistor-dil:4R-N0603-ARC
Connections:
- net GND: now also RN11A.1, RN11A.2, RN11B.1
- net TCK: now also RN11B.2
- net TDI: now also RN11D.2
- net TMS: now also RN11C.2
- net VCCIO: now also RN11C.1, RN11D.1

Commit message: Add files via upload
Parts:
- added R26: 10, rcl:R-EU_R0805
Connections:
- removed net ALE: U1.IO24, U13.EN
- new net ALE_FPGA: R26.1, U1.IO24
- new net N$6: R26.2, U13.EN
Changed lines of the file:
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@@
 <setting verticaltext="up"/>
 </settings>
-<grid distance="0.1" unitdist="inch" unit="inch" style="lines" multiple="1" display="no" altdistance="0.01" altunitdist="inch" altunit="inch"/>
+<grid distance="0.1" unitdist="inch" unit="inch" style="lines" multiple="1" display="yes" altdistance="0.01" altunitdist="inch" altunit="inch"/>
 <layers>
-<layer number="1" name="Top" color="4" fill="1" visible="yes" active="no"/>
-<layer number="2" name="Route2" color="16" fill="1" visible="yes" active="no"/>
-<layer number="3" name="Route3" color="17" fill="1" visible="yes" active="no"/>
-<layer number="4" name="Route4" color="18" fill="1" visible="yes" active="no"/>
-<layer number="5" name="Route5" color="19" fill="1" visible="yes" active="no"/>
-<layer number="6" name="Route6" color="25" fill="1" visible="yes" active="no"/>
-<layer number="7" name="Route7" color="26" fill="1" visible="yes" active="no"/>
-<layer number="8" name="Route8" color="27" fill="1" visible="yes" active="no"/>
-<layer number="9" name="Route9" color="28" fill="1" visible="yes" active="no"/>
-<layer number="10" name="Route10" color="29" fill="1" visible="yes" active="no"/>
-<layer number="11" name="Route11" color="30" fill="1" visible="yes" active="no"/>
-<layer number="12" name="Route12" color="20" fill="1" visible="yes" active="no"/>
-<layer number="13" name="Route13" color="21" fill="1" visible="yes" active="no"/>
-<layer number="14" name="Route14" color="22" fill="1" visible="yes" active="no"/>
-<layer number="15" name="Route15" color="23" fill="1" visible="yes" active="no"/>
-<layer number="16" name="Bottom" color="1" fill="1" visible="yes" active="no"/>
-<layer number="17" name="Pads" color="2" fill="1" visible="yes" active="no"/>
-<layer number="18" name="Vias" color="2" fill="1" visible="yes" active="no"/>
-<layer number="19" name="Unrouted" color="6" fill="1" visible="yes" active="no"/>
-<layer number="20" name="Dimension" color="15" fill="1" visible="yes" active="no"/>
-<layer number="21" name="tPlace" color="7" fill="1" visible="yes" active="no"/>
-<layer number="22" name="bPlace" color="7" fill="1" visible="yes" active="no"/>
-<layer number="23" name="tOrigins" color="15" fill="1" visible="yes" active="no"/>
-<layer number="24" name="bOrigins" color="15" fill="1" visible="yes" active="no"/>
-<layer number="25" name="tNames" color="7" fill="1" visible="yes" active="no"/>
-<layer number="26" name="bNames" color="7" fill="1" visible="yes" active="no"/>
-<layer number="27" name="tValues" color="7" fill="1" visible="yes" active="no"/>
-<layer number="28" name="bValues" color="7" fill="1" visible="yes" active="no"/>
+<layer number="1" name="Top" color="4" fill="1" visible="no" active="no"/>
+<layer number="2" name="Route2" color="16" fill="1" visible="no" active="no"/>
+<layer number="3" name="Route3" color="17" fill="1" visible="no" active="no"/>
+<layer number="4" name="Route4" color="18" fill="1" visible="no" active="no"/>
+<layer number="5" name="Route5" color="19" fill="1" visible="no" active="no"/>
+<layer number="6" name="Route6" color="25" fill="1" visible="no" active="no"/>
+<layer number="7" name="Route7" color="26" fill="1" visible="no" active="no"/>
+<layer number="8" name="Route8" color="27" fill="1" visible="no" active="no"/>
+<layer number="9" name="Route9" color="28" fill="1" visible="no" active="no"/>
+<layer number="10" name="Route10" color="29" fill="1" visible="no" active="no"/>
+<layer number="11" name="Route11" color="30" fill="1" visible="no" active="no"/>
+<layer number="12" name="Route12" color="20" fill="1" visible="no" active="no"/>
+<layer number="13" name="Route13" color="21" fill="1" visible="no" active="no"/>
+<layer number="14" name="Route14" color="22" fill="1" visible="no" active="no"/>
+<layer number="15" name="Route15" color="23" fill="1" visible="no" active="no"/>
+<layer number="16" name="Bottom" color="1" fill="1" visible="no" active="no"/>
+<layer number="17" name="Pads" color="2" fill="1" visible="no" active="no"/>
+<layer number="18" name="Vias" color="2" fill="1" visible="no" active="no"/>
+<layer number="19" name="Unrouted" color="6" fill="1" visible="no" active="no"/>
+<layer number="20" name="Dimension" color="15" fill="1" visible="no" active="no"/>
+<layer number="21" name="tPlace" color="7" fill="1" visible="no" active="no"/>
+<layer number="22" name="bPlace" color="7" fill="1" visible="no" active="no"/>
+<layer number="23" name="tOrigins" color="15" fill="1" visible="no" active="no"/>
+<layer number="24" name="bOrigins" color="15" fill="1" visible="no" active="no"/>
+<layer number="25" name="tNames" color="7" fill="1" visible="no" active="no"/>
+<layer number="26" name="bNames" color="7" fill="1" visible="no" active="no"/>
+<layer number="27" name="tValues" color="7" fill="1" visible="no" active="no"/>
+<layer number="28" name="bValues" color="7" fill="1" visible="no" active="no"/>
 <layer number="29" name="tStop" color="7" fill="3" visible="no" active="no"/>
 <layer number="30" name="bStop" color="7" fill="6" visible="no" active="no"/>
@@
 <layer number="35" name="tGlue" color="7" fill="4" visible="no" active="no"/>
 <layer number="36" name="bGlue" color="7" fill="5" visible="no" active="no"/>
-<layer number="37" name="tTest" color="7" fill="1" visible="yes" active="no"/>
-<layer number="38" name="bTest" color="7" fill="1" visible="yes" active="no"/>
+<layer number="37" name="tTest" color="7" fill="1" visible="no" active="no"/>
+<layer number="38" name="bTest" color="7" fill="1" visible="no" active="no"/>
 <layer number="39" name="tKeepout" color="4" fill="11" visible="no" active="no"/>
 <layer number="40" name="bKeepout" color="1" fill="11" visible="no" active="no"/>
@@
 <layer number="44" name="Drills" color="7" fill="1" visible="no" active="no"/>
 <layer number="45" name="Holes" color="7" fill="1" visible="no" active="no"/>
-<layer number="46" name="Milling" color="3" fill="1" visible="yes" active="no"/>
-<layer number="47" name="Measures" color="7" fill="1" visible="yes" active="no"/>
-<layer number="48" name="Document" color="7" fill="1" visible="yes" active="no"/>
-<layer number="49" name="Reference" color="7" fill="1" visible="yes" active="no"/>
-<layer number="50" name="dxf" color="7" fill="1" visible="yes" active="no"/>
-<layer number="51" name="tDocu" color="7" fill="1" visible="yes" active="no"/>
-<layer number="52" name="bDocu" color="7" fill="1" visible="yes" active="no"/>
-<layer number="56" name="wert" color="7" fill="1" visible="yes" active="no"/>
+<layer number="46" name="Milling" color="3" fill="1" visible="no" active="no"/>
+<layer number="47" name="Measures" color="7" fill="1" visible="no" active="no"/>
+<layer number="48" name="Document" color="7" fill="1" visible="no" active="no"/>
+<layer number="49" name="Reference" color="7" fill="1" visible="no" active="no"/>
+<layer number="50" name="dxf" color="7" fill="1" visible="no" active="no"/>
+<layer number="51" name="tDocu" color="7" fill="1" visible="no" active="no"/>
+<layer number="52" name="bDocu" color="7" fill="1" visible="no" active="no"/>
+<layer number="56" name="wert" color="7" fill="1" visible="no" active="no"/>
 <layer number="88" name="SimResults" color="9" fill="1" visible="yes" active="yes"/>
 <layer number="89" name="SimProbes" color="9" fill="1" visible="yes" active="yes"/>
@@
 <part name="GND81" library="supply1" library_urn="urn:adsk.eagle:library:371" deviceset="GND" device=""/>
 <part name="VCC15" library="supply1" library_urn="urn:adsk.eagle:library:371" deviceset="VCCIO" device=""/>
+<part name="R26" library="rcl" library_urn="urn:adsk.eagle:library:334" deviceset="R-EU_" device="R0805" package3d_urn="urn:adsk.eagle:package:23553/2" value="10"/>
 </parts>
 <sheets>
@@
 <attribute name="VALUE" x="29.718" y="158.242" size="1.778" layer="96" rot="MR180"/>
 </instance>
+<instance part="R26" gate="G$1" x="-236.22" y="60.96" smashed="yes">
+<attribute name="NAME" x="-236.648" y="64.3626" size="1.778" layer="95" rot="R180"/>
+<attribute name="VALUE" x="-232.068" y="64.368" size="1.778" layer="96" rot="R180"/>
+</instance>
 </instances>
 <busses>
@@
 </segment>
 </net>
-<net name="ALE" class="0">
-<segment>
-<wire x1="10.16" y1="-48.26" x2="10.16" y2="-63.5" width="0.1524" layer="91"/>
-<label x="10.16" y="-62.484" size="1.778" layer="95" rot="R90"/>
-<pinref part="U1" gate="G$1" pin="IO24"/>
-</segment>
-<segment>
-<wire x1="-205.74" y1="60.96" x2="-213.36" y2="60.96" width="0.1524" layer="91"/>
-<label x="-213.36" y="60.96" size="1.778" layer="95"/>
-<pinref part="U13" gate="G$1" pin="EN"/>
-</segment>
-</net>
 <net name="N$17" class="0">
 <segment>
@@
 </segment>
 </net>
+<net name="ALE_FPGA" class="0">
+<segment>
+<wire x1="10.16" y1="-48.26" x2="10.16" y2="-63.5" width="0.1524" layer="91"/>
+<label x="10.16" y="-62.484" size="1.778" layer="95" rot="R90"/>
+<pinref part="U1" gate="G$1" pin="IO24"/>
+</segment>
+<segment>
+<pinref part="R26" gate="G$1" pin="1"/>
+<wire x1="-241.3" y1="60.96" x2="-259.08" y2="60.96" width="0.1524" layer="91"/>
+<label x="-256.54" y="60.96" size="1.778" layer="95"/>
+</segment>
+</net>
+<net name="N$6" class="0">
+<segment>
+<pinref part="U13" gate="G$1" pin="EN"/>
+<pinref part="R26" gate="G$1" pin="2"/>
+<wire x1="-205.74" y1="60.96" x2="-231.14" y2="60.96" width="0.1524" layer="91"/>
+</segment>
+</net>
