File: PCB/FPGA_DENDY_SE.sch (EAGLE design)
At the start: 141 parts, among them CN1 DENDY60PINSLOT, J1 /PAL, J2 /DENDY, Q1 14.318 MHz, Q2 17.734 MHz, U1 EP1C3T100C8N, U10 SN74LVC1G125DBVR, U11 SN74LVC1G240DBVR, U12 SN74LVC1G240DBVR, U13 SN74LVC1G240DBVR, U14 SN74LVC1G240DBVR, U15 OPA2134U, U2 SN74LVC8T245, U3 74LS373WMSO20, U4 SN74LVC8T245, U5 SN74LVC2G34DBVR, U6 74LVC1G04GV, U7 EPCS4, U8 SN74LVC1G3157, U9 THS7314DR, X1 057-010-1, X2 JOYPAD1, X3 9V, X4 JOYPAD2

Commit message: Add files via upload
Parts:
- added JP2: CLK_EXT, pinhead:PINHD-1X1
- added JP4: AUDIO, pinhead:PINHD-1X3
- added JP5: VIDEO, pinhead:PINHD-1X3
- R23: value 2k -> 4k7
- R25: value 4k7 -> 2k
Connections:
- removed net CLK_EXT: R10.2
- removed net VIDEO: C44.-
- new net N$3: JP2.1, R10.2
- new net N$45: C44.-, JP5.2
- net +5V: now also C7.1; no longer C7.2
- net GND: now also C7.2, JP4.1, JP5.1, JP5.3; no longer C7.1
- net LCH: now also JP4.3
- net RCH: now also JP4.2
- net SND: now also R23.1; no longer R25.1
- net SND_EXT: now also R25.1; no longer R23.1
Other:
- moved on the sheet: C48, C49, C5, C50, C51, C6, C7, R10, R2, R23, R24, R25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

Commit message: Add files via upload
Parts:
- removed JP3: #RESET, jumper:JP4QE
- removed Q1: 14.318 MHz, crystal-geyer_V1_0:KXO-PXO/XO-V97
- removed Q2: 17.734 MHz, crystal-geyer_V1_0:KXO-PXO/XO-V95
- added J3: #RESET, jumper:JP1E
- added XO1: 14.318 MHz, crystal-geyer_V1_0:KXO-PXO/XO-V97
- added XO2: 17.734 MHz, crystal-geyer_V1_0:KXO-PXO/XO-V95
Connections:
- net /RESET: now also J3.1; no longer JP3-1.1
- net GND: now also J3.2, XO1.GND, XO2.GND; no longer JP3-1.2, Q1.GND, Q2.GND
- net N$17: now also XO1.OUT; no longer Q1.OUT
- net N$18: now also XO2.OUT; no longer Q2.OUT
- net VCCINT: now also C24.1, C25.1; no longer C22.2, C23.2
- net VCCIO: now also C22.2, C23.2, XO1.VDD, XO2.VDD; no longer C24.1, C25.1, Q1.VDD, Q2.VDD
Other:
- moved on the sheet: C1, C14, C15, C16, C17, C18, C19, C2, C22, C23, C24, C25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

Commit message: Add files via upload
Parts:
- U2, U4: device SnapEDA-Library:SN74LVC8T245 -> SN74LVC8T245:SN74LVC8T245
Connections:
- net +5V: now also C6.1, U4.VCCA; no longer C7.1, U4.VCCB@1, U4.VCCB@2
- net VCCIO: now also C7.1, U4.VCCB@1, U4.VCCB@2; no longer C6.1, U4.VCCA
Other:
- moved on the sheet: C3, C4, C6, C7, RN5A, RN5B, RN5C, RN5D, RN6A, RN6B, RN6C, RN6D
